Commit message: auto(2026-07-18_14:29:20): assets/piper/piper_dual_description.urdf, assets/piper/piper_dual.xml, assets/piper/scene_dual.xml, piper_pico/config.py, piper_pico/real/real_piper_teleop_controller.py, +3 more

File: assets/piper/piper_dual_description.urdf (robot description, URDF)
Before this commit: robot piper_dual, 21 links, 20 joints
Joints:
- joint base_to_left_base: origin xyz=0 -0.18 0.72 rpy=0 0 0 -> xyz=0 0.18 0.72 rpy=0 0 0
- joint base_to_right_base: origin xyz=0 0.18 0.72 rpy=0 0 0 -> xyz=0 -0.18 0.72 rpy=0 0 0
